File: KiCad/MicroFlight/MicroESC1S3mosfets.sch (KiCad schematic (older format))
At the start: 19 parts, among them J1 C2CK, J2 C2D, J3 A, J4 B, J5 C, Q1 DUAL_NP, Q2 DUAL_NP, Q3 DUAL_NP, U5 EFM8BB21

Commit message: PCB - added optional shunt for current sensing
Parts:
- removed J3: A, Pin_Headers:Pin_Header_Straight_1x01_Pitch1.27mm, symbol Connector_Generic:Conn_01x01
- removed J4: B, Pin_Headers:Pin_Header_Straight_1x01_Pitch1.27mm, symbol Connector_Generic:Conn_01x01
- removed J5: C, Pin_Headers:Pin_Header_Straight_1x01_Pitch1.27mm, symbol Connector_Generic:Conn_01x01
- added J3: MOTOR, Connectors_Molex:Molex_PicoBlade_53047-0310_03x1.25mm_Straight, symbol Connector_Generic:Conn_01x03
Connections:
- wire segments 100 -> 103
Changed lines of the file:
@@
 Connection ~ 8750 3550
 Connection ~ 9050 5050
-$Comp
-L Connector_Generic:Conn_01x01 J3
-U 1 1 59A81331
-P 9500 2050
-F 0 "J3" H 9500 2150 50  0000 C CNN
-F 1 "A" H 9500 1950 50  0000 C CNN
-F 2 "Pin_Headers:Pin_Header_Straight_1x01_Pitch1.27mm" H 9500 2050 50  0001 C CNN
-F 3 "" H 9500 2050 50  0001 C CNN
-	1    9500 2050
-	1    0    0    -1
-$EndComp
-$Comp
-L Connector_Generic:Conn_01x01 J4
-U 1 1 59A81397
-P 9500 3550
-F 0 "J4" H 9500 3650 50  0000 C CNN
-F 1 "B" H 9500 3450 50  0000 C CNN
-F 2 "Pin_Headers:Pin_Header_Straight_1x01_Pitch1.27mm" H 9500 3550 50  0001 C CNN
-F 3 "" H 9500 3550 50  0001 C CNN
-	1    9500 3550
-	1    0    0    -1
-$EndComp
-$Comp
-L Connector_Generic:Conn_01x01 J5
-U 1 1 59A81475
-P 9500 5050
-F 0 "J5" H 9500 5150 50  0000 C CNN
-F 1 "C" H 9500 4950 50  0000 C CNN
-F 2 "Pin_Headers:Pin_Header_Straight_1x01_Pitch1.27mm" H 9500 5050 50  0001 C CNN
-F 3 "" H 9500 5050 50  0001 C CNN
-	1    9500 5050
-	1    0    0    -1
-$EndComp
 Wire Wire Line
 	1400 2250 4000 2250
@@
 Text Label 6700 1950 0    50   ~ 0
 Mpwr
+$Comp
+L Connector_Generic:Conn_01x03 J3
+U 1 1 5DF9C5F3
+P 10100 2850
+F 0 "J3" H 10180 2892 50  0000 L CNN
+F 1 "MOTOR" H 10180 2801 50  0000 L CNN
+F 2 "Connectors_Molex:Molex_PicoBlade_53047-0310_03x1.25mm_Straight" H 10100 2850 50  0001 C CNN
+F 3 "~" H 10100 2850 50  0001 C CNN
+	1    10100 2850
+	1    0    0    -1
+$EndComp
+Wire Wire Line
+	9900 2750 9650 2750
+Wire Wire Line
+	9900 2850 9650 2850
+Wire Wire Line
+	9900 2950 9650 2950
+Text Label 9650 2750 0    50   ~ 0
+M_A
+Text Label 9650 2850 0    50   ~ 0
+M_B
+Text Label 9650 2950 0    50   ~ 0
+M_C
 $EndSCHEMATC
