File: KiCad/MicroFlight/MicroFlight.sch (KiCad schematic (older format))
At the start: 46 parts, among them J10 SRV3, J6 BIND, J7 BAT, J8 SRV1, J9 SRV2, U1 TPS61222, U2 ATmega328P-AU, U3 RT9013-33, U4 CC2500, Y1 16MHZ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

Commit message: PCB - added optional shunt for current sensing
Parts:
- added R13: 0.022, Resistors_SMD:R_1206, symbol Device:R
- added R14: 0.022, Resistors_SMD:R_2010, symbol Device:R
- added U6: MAX9610, TO_SOT_Packages_SMD:SOT-353_SC-70-5, symbol KiCadCustomLibraries:MAX9610
Connections:
- net +BATT: now also R13.1, R14.1, U6.4 (RS-); no longer J7.2 (Pin_2)
- net A2: now also U6.3 (OUT); no longer R1.1, R2.2
- net GND: now also U6.1 (GND), U6.2 (GND)
- net A1: now reaches U2.19 (ADC6)
- net A1: now also R1.1, R2.2
- new net: J7.2 (Pin_2), R13.2, R14.2, U6.5 (RS+)
- no-connect marks 12 -> 11
Other:
- moved on the sheet: C1, C3, C5, C7, J7, L1, U1, U3
